File: Board design/openinduction main board.kicad_sch (KiCad schematic)
At the start: 22 parts, among them Q1 NMOS, T1 Transformer_1P_2S, U1 UCC28704DBV

Commit message: kajdkajs
Parts:
- added C1: C_Polarized, symbol Device:C_Polarized
- added D2: B40C3x00-2200A, Diode_THT:Diode_Bridge_32.0x5.6x17.0mm_P10.0mm_P7.5mm, symbol Diode_Bridge:B40C3x00-2200A
Other:
- moved on the sheet: C2, C3, Cout, Csnub, D1, D3, D4, Dsnub2, Q1, R1, R2, R3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

Commit message: jaskjhaskjdahskjdhdslkahdblhfs
Connections:
- net +12V: now also C1.2, D2.1 (-)
- net VS: now also C1.1, D2.4 (+)
- net AC: now reaches D2.2
- net NEUT: now reaches D2.3
Other:
- moved on the sheet: C1, D2

Commit message: added todo and updated main board to add connectors
Parts:
- added J1, J2, J3, J4: Conn_01x01_Pin, symbol Connector:Conn_01x01_Pin
Connections:
- net +12V: now also J3.1 (Pin_1); no longer C1.2, C2.2, C3.2, Cout.2, D2.1 (-), D3.2 (A), R2.2, R8.2, Rbld.2, T1.1 (AA), T1.4 (SB), U1.1 (GND)
- net VS: now also J2.1 (Pin_1)
- new net GND: C1.2, C2.2, C3.2, Cout.2, D2.1 (-), D3.2 (A), J1.1 (Pin_1), R2.2, R8.2, Rbld.2, T1.1 (AA), T1.4 (SB), U1.1 (GND)
Other:
- note added: "change vs to +200v"
- note added: "to do: change symbol names find components do footprints add power connectors to connect to nick's board"
- note removed: "to do: change symbol names find components do footprints"
- moved on the sheet: C1, D2
