File: Board design/inverterBoard.kicad_sch (KiCad schematic)
At the start: 13 parts, among them Q1 IRF740, Q7 IRF740, U1 ESP32-S2, U2 FAN7842

Commit message: added updated datasheets and connectors to inverterBoard
Parts:
- removed D1, D2: D_Schottky, symbol Device:D_Schottky
- removed L1: L, symbol Device:L
- added J1, J2, J3, J4, J5: Conn_01x01_Pin, symbol Connector:Conn_01x01_Pin
- R1, R2: footprint (none) -> Resistor_THT:R_Axial_DIN0411_L9.9mm_D3.6mm_P20.32mm_Horizontal
Connections:
- net GND: now also J3.1 (Pin_1)
- net at C1.1, L2.1: now also J1.1 (Pin_1)
- new net +12V: J4.1 (Pin_1)
- new net +200v: J5.1 (Pin_1)
- new net +5v: J2.1 (Pin_1)
Other:
- note added: "add dc cap to mcc input and input of vdd of u2"
- note added: "be able to handle ac have enough microferrets for the oscillator to oscillate with the proper range and find what cap value for the circuit will do so"
- note added: "c1 needs to"
- moved on the sheet: C1
